Commit message: simulation and move robot

File: rover_description/urdf/depth_camera.xacro (robot description, xacro)
@@ -1,47 +1,59 @@
 <?xml version="1.0"?>
-<robot xmlns:xacro="http://www.ros.org/wiki/xacro" >
-    <joint name="camera_joint" type="fixed">
-        <parent link="body"/>
-        <child link="camera_link"/>
-        <origin xyz="0.3 0 0.25" rpy="0 0 0"/>
-    </joint>
-    <link name="camera_link">
-        <visual>
-            <geometry>
-                <box size="0.02 0.075 0.03"/>
-            </geometry>
-            <material name="red"/>
-        </visual>
-    </link>
-    <joint name="camera_optical_joint" type="fixed">
-        <parent link="camera_link"/>
-        <child link="camera_link_optical"/>
-        <origin xyz="0 0 0" rpy="${-pi/2} 0 ${-pi/2}"/>
-    </joint>
-    <link name="camera_link_optical"></link>
-    <gazebo reference="camera_link">
-        <material>Gazebo/Red</material>
-        <sensor name="camera" type="depth">
-            <pose> 0 0 0 0 0 0 </pose>
-            <visualize>true</visualize>
-            <update_rate>10</update_rate>
-            <camera>
-                <horizontal_fov>1.089</horizontal_fov>
-                <image>
-                    <format>B8G8R8</format>
-                    <width>640</width>
-                    <height>480</height>
-                </image>
-                <clip>
-                    <near>0.05</near>
-                    <far>8.0</far>
-                </clip>
-            </camera>
-            <plugin name="camera_controller" filename="libgazebo_ros_camera.so">
-                <frame_name>camera_link_optical</frame_name>
-                <min_depth>0.1</min_depth>
-                <max_depth>100.0</max_depth>
-            </plugin>
-        </sensor>
-    </gazebo>
+<robot xmlns:xacro="http://www.ros.org/wiki/xacro">
+  <!-- Fixed joint to mount camera on robot body -->
+  <joint name="camera_joint" type="fixed">
+    <parent link="body"/>
+    <child link="camera_link"/>
+    <origin xyz="0.3 0 0.25" rpy="0 0 0"/>
+  </joint>
+  <!-- Camera housing link -->
+  <link name="camera_link">
+    <visual>
+      <geometry>
+        <box size="0.02 0.075 0.03"/>
+      </geometry>
+      <material name="red">
+        <color rgba="1 0 0 1"/>
+      </material>
+    </visual>
+    <collision>
+      <geometry>
+        <box size="0.02 0.075 0.03"/>
+      </geometry>
+    </collision>
+    <inertial>
+      <mass value="0.1"/>
+      <inertia ixx="1e-4" iyy="1e-4" izz="1e-4" ixy="0" ixz="0" iyz="0"/>
+    </inertial>
+  </link>
+  <!-- Optical frame (REP-103: Z forward, X right, Y down) -->
+  <joint name="camera_optical_joint" type="fixed">
+    <parent link="camera_link"/>
+    <child link="camera_optical_frame"/>
+    <origin xyz="0 0 0" rpy="${-pi/2} 0 ${-pi/2}"/>
+  </joint>
+  <link name="camera_optical_frame"/>
+  <gazebo reference="camera_link">
+    <material>Gazebo/Black</material>
+    <sensor name="camera" type="camera">
+        <pose> 0 0 0 0 0 0 </pose>
+        <visualize>true</visualize>
+        <update_rate>10</update_rate>
+        <camera>
+            <camera_info_topic>camera/camera_info</camera_info_topic>
+            <horizontal_fov>1.089</horizontal_fov>
+            <image>
+                <format>R8G8B8</format>
+                <width>640</width>
+                <height>480</height>
+            </image>
+            <clip>
+                <near>0.05</near>
+                <far>8.0</far>
+            </clip>
+        </camera>
+        <topic>camera/image_raw</topic>
+        <gz_frame_id>camera_link_optical</gz_frame_id>
+    </sensor>
+</gazebo>
 </robot>

File: rover_description/urdf/robot.urdf.xacro (robot description, xacro)
@@ -1,6 +1,6 @@
 <?xml version="1.0"?>
-<robot xmlns:xacro="http://www.ros.org/wiki/xacro"  name="robot">
-    <xacro:arg name="use_ros2_control" default="true"/>
-    <xacro:arg name="sim_mode" default="false"/>
+<robot xmlns:xacro="http://www.ros.org/wiki/xacro" name="robot">
+    <xacro:arg name="use_ros2_control" default="true" />
+    <xacro:arg name="sim_mode" default="false" />
     <xacro:include filename="main.xacro" />
     <!-- <xacro:if value="$(arg use_ros2_control)">
@@ -11,5 +11,5 @@
     </xacro:unless> -->
     <xacro:include filename="lidar.xacro" />
-     <!-- <xacro:include filename="camera.xacro" /> -->
+    <!-- <xacro:include filename="camera.xacro" /> -->
     <xacro:include filename="depth_camera.xacro" />
 </robot>

File: rover_description/urdf/simple_main.xacro (robot description, xacro)
@@ -220,53 +220,4 @@
         <material>Gazebo/Blue</material>
     </gazebo>
-    <!-- PL,ATFORM LINK -->
-    <joint name="platform_joint" type="fixed">
-        <parent link="base_link" />
-        <child link="platform" />
-        <origin xyz="0 0 ${(chassis_height)}" />
-    </joint>
-    <link name="platform">
-        <visual>
-            <origin xyz="${platform_length/2} 0 ${platform_height/2}" />
-            <geometry>
-                <box size="${platform_length} ${platform_width} ${platform_height}" />
-            </geometry>
-            <material name="pink" />
-        </visual>
-        <collision>
-            <origin xyz="${platform_length/2} 0 ${platform_height/2}" />
-            <geometry>
-                <box size="${platform_length} ${platform_width} ${platform_height}" />
-            </geometry>
-        </collision>
-        <xacro:inertial_box mass="0.5" x="${platform_length}" y="${platform_width}"
-            z="${platform_height}">
-            <origin xyz="${platform_length/2} 0 ${platform_height/2}" rpy="0 0 0" />
-        </xacro:inertial_box>
-    </link>
-    <!-- BODY LINK -->
-    <joint name="body_joint" type="fixed">
-        <parent link="base_link" />
-        <child link="body" />
-        <origin xyz="0.3 0 ${(chassis_height)}" />
-    </joint>
-    <link name="body">
-        <visual>
-            <origin xyz="${body_length/2} 0 ${body_height/2}" />
-            <geometry>
-                <box size="${body_length} ${body_width} ${body_height}" />
-            </geometry>
-            <material name="yellow" />
-        </visual>
-        <collision>
-            <origin xyz="${body_length/2} 0 ${body_height/2}" />
-            <geometry>
-                <box size="${body_length} ${body_width} ${body_height}" />
-            </geometry>
-        </collision>
-        <xacro:inertial_box mass="0.5" x="${body_length}" y="${body_width}" z="${body_height}">
-            <origin xyz="${body_length/2} 0 ${body_height/2}" rpy="0 0 0" />
-        </xacro:inertial_box>
-    </link>
     <gazebo>
         <plugin
