Commit message: feat: AgriBot V2 robot, hillside terrain, and simulation fixes
Robot (rover_description):
- Add robot_v2.urdf.xacro / main_v2.xacro — redesigned robot with larger
  wheels (r=0.10 m), wider 0.66 m track, 3-sided cargo bed with retaining
  walls, front bumper, and a xacro wheel macro to eliminate code duplication
- Fix DiffDrive plugin to drive all 4 wheels (was rear-only)
- Fix odom topic mismatch (odom/unfiltered → odom)
- Add missing JointStatePublisher Gazebo plugin
- Fix depth_camera gz_frame_id (camera_link_optical → camera_optical_frame)
- Fix skid_steer.urdf.xacro XML namespace (missing www.)
- Add wheel friction (μ=0.9) to all four wheels for slope traction
- Add Gazebo material tags for platform and body links

World / simulation (world_simulation):
- Replace flat grass patches with procedurally generated 40×40 m hillside
  terrain (8 m elevation, ~15 % grade) via heightmap model
- Add hill_terrain model with collision friction (μ=0.85) tuned for slopes
- Add generate_heightmap.py script (257×257 grayscale PNG, S-curve slope)
- Add gazebo.launch.py — robot in empty world for quick testing
- Fix sim.launch.py: remove conflicting joint_state_publisher node, remove
  non-existent GZ_SIM_PLUGIN_PATH, spawn robot at hilltop with 5 s delay,
  switch to robot_v2.urdf.xacro
- Fix grass_world.sdf: embed terrain inline (avoids model:// URI failure),
  remove __default__ normal-map URIs that caused world-load crash

Docs:
- Rewrite README for AgriSpark Hackathon 2025 "Hack the Hills" submission
  with problem statement, solution overview, V1→V2 comparison table, and
  roadmap

Co-Authored-By: Claude Sonnet 4.6 <noreply@anthropic.com>

File: rover_description/urdf/depth_camera.xacro (robot description, xacro)
@@ -54,5 +54,5 @@
         </camera>
         <topic>camera/image_raw</topic>
-        <gz_frame_id>camera_link_optical</gz_frame_id>
+        <gz_frame_id>camera_optical_frame</gz_frame_id>
     </sensor>
 </gazebo>

File: rover_description/urdf/main.xacro (robot description, xacro)
@@ -140,4 +140,8 @@
     <gazebo reference="front_left_wheel">
         <material>Gazebo/Blue</material>
+        <mu1>0.9</mu1>
+        <mu2>0.9</mu2>
+        <slip1>0.0</slip1>
+        <slip2>0.0</slip2>
     </gazebo>
     <joint name="rear_left_wheel_joint" type="continuous">
@@ -166,4 +170,8 @@
     <gazebo reference="rear_left_wheel">
         <material>Gazebo/Blue</material>
+        <mu1>0.9</mu1>
+        <mu2>0.9</mu2>
+        <slip1>0.0</slip1>
+        <slip2>0.0</slip2>
     </gazebo>
     <!-- RIGHT WHEEL LINK -->
@@ -193,4 +201,8 @@
     <gazebo reference="front_right_wheel">
         <material>Gazebo/Blue</material>
+        <mu1>0.9</mu1>
+        <mu2>0.9</mu2>
+        <slip1>0.0</slip1>
+        <slip2>0.0</slip2>
     </gazebo>
     <joint name="rear_right_wheel_joint" type="continuous">
@@ -219,4 +231,8 @@
     <gazebo reference="rear_right_wheel">
         <material>Gazebo/Blue</material>
+        <mu1>0.9</mu1>
+        <mu2>0.9</mu2>
+        <slip1>0.0</slip1>
+        <slip2>0.0</slip2>
     </gazebo>
     <!-- PL,ATFORM LINK -->
@@ -269,25 +285,41 @@
         </xacro:inertial_box>
     </link>
+    <gazebo reference="platform">
+        <material>Gazebo/Pink</material>
+    </gazebo>
+    <gazebo reference="body">
+        <material>Gazebo/Yellow</material>
+    </gazebo>
     <gazebo>
-        <plugin
-        filename="gz-sim-diff-drive-system"
-        name="gz::sim::systems::DiffDrive">
+        <plugin filename="gz-sim-diff-drive-system" name="gz::sim::systems::DiffDrive">
             <topic>cmd_vel</topic>
-            <!-- <frame_id>odom</frame_id> -->
             <child_frame_id>base_footprint</child_frame_id>
-            <odom_topic>odom/unfiltered</odom_topic>
-            <!-- <tf_topic>/tf</tf_topic> -->
-        <left_joint>rear_left_wheel_joint</left_joint>
-        <right_joint>rear_right_wheel_joint</right_joint>
-            <wheel_separation>0.45</wheel_separation>
+            <odom_topic>odom</odom_topic>
+            <left_joint>front_left_wheel_joint</left_joint>
+            <right_joint>front_right_wheel_joint</right_joint>
+            <left_joint>rear_left_wheel_joint</left_joint>
+            <right_joint>rear_right_wheel_joint</right_joint>
+            <wheel_separation>${2 * wheel_offset_y}</wheel_separation>
             <wheel_radius>${wheel_radius}</wheel_radius>
-        <max_linear_acceleration>1</max_linear_acceleration>
-        <min_linear_acceleration>-1</min_linear_acceleration>
-        <max_angular_acceleration>2</max_angular_acceleration>
-        <min_angular_acceleration>-2</min_angular_acceleration>
-        <max_linear_velocity>0.5</max_linear_velocity>
-        <min_linear_velocity>-0.5</min_linear_velocity>
-        <max_angular_velocity>1</max_angular_velocity>
-        <min_angular_velocity>-1</min_angular_velocity>        </plugin>
-      </gazebo>
+            <max_linear_acceleration>1</max_linear_acceleration>
+            <min_linear_acceleration>-1</min_linear_acceleration>
+            <max_angular_acceleration>2</max_angular_acceleration>
+            <min_angular_acceleration>-2</min_angular_acceleration>
+            <max_linear_velocity>0.5</max_linear_velocity>
+            <min_linear_velocity>-0.5</min_linear_velocity>
+            <max_angular_velocity>1</max_angular_velocity>
+            <min_angular_velocity>-1</min_angular_velocity>
+        </plugin>
+    </gazebo>
+    <gazebo>
+        <plugin filename="gz-sim-joint-state-publisher-system"
+            name="gz::sim::systems::JointStatePublisher">
+            <topic>joint_states</topic>
+            <update_rate>50</update_rate>
+            <joint_name>front_left_wheel_joint</joint_name>
+            <joint_name>front_right_wheel_joint</joint_name>
+            <joint_name>rear_left_wheel_joint</joint_name>
+            <joint_name>rear_right_wheel_joint</joint_name>
+        </plugin>
+    </gazebo>
 </robot>

File: rover_description/urdf/simple_main.xacro (robot description, xacro)
@@ -221,24 +221,34 @@
     </gazebo>
     <gazebo>
-        <plugin
-        filename="gz-sim-diff-drive-system"
-        name="gz::sim::systems::DiffDrive">
+        <plugin filename="gz-sim-diff-drive-system" name="gz::sim::systems::DiffDrive">
             <topic>cmd_vel</topic>
-            <!-- <frame_id>odom</frame_id> -->
             <child_frame_id>base_footprint</child_frame_id>
-            <odom_topic>odom/unfiltered</odom_topic>
-            <!-- <tf_topic>/tf</tf_topic> -->
-        <left_joint>rear_left_wheel_joint</left_joint>
-        <right_joint>rear_right_wheel_joint</right_joint>
-            <wheel_separation>0.45</wheel_separation>
+            <odom_topic>odom</odom_topic>
+            <left_joint>front_left_wheel_joint</left_joint>
+            <right_joint>front_right_wheel_joint</right_joint>
+            <left_joint>rear_left_wheel_joint</left_joint>
+            <right_joint>rear_right_wheel_joint</right_joint>
+            <wheel_separation>${2 * wheel_offset_y}</wheel_separation>
             <wheel_radius>${wheel_radius}</wheel_radius>
-        <max_linear_acceleration>1</max_linear_acceleration>
-        <min_linear_acceleration>-1</min_linear_acceleration>
-        <max_angular_acceleration>2</max_angular_acceleration>
-        <min_angular_acceleration>-2</min_angular_acceleration>
-        <max_linear_velocity>0.5</max_linear_velocity>
-        <min_linear_velocity>-0.5</min_linear_velocity>
-        <max_angular_velocity>1</max_angular_velocity>
-        <min_angular_velocity>-1</min_angular_velocity>        </plugin>
-      </gazebo>
+            <max_linear_acceleration>1</max_linear_acceleration>
+            <min_linear_acceleration>-1</min_linear_acceleration>
+            <max_angular_acceleration>2</max_angular_acceleration>
+            <min_angular_acceleration>-2</min_angular_acceleration>
+            <max_linear_velocity>0.5</max_linear_velocity>
+            <min_linear_velocity>-0.5</min_linear_velocity>
+            <max_angular_velocity>1</max_angular_velocity>
+            <min_angular_velocity>-1</min_angular_velocity>
+        </plugin>
+    </gazebo>
+    <gazebo>
+        <plugin filename="gz-sim-joint-state-publisher-system"
+            name="gz::sim::systems::JointStatePublisher">
+            <topic>joint_states</topic>
+            <update_rate>50</update_rate>
+            <joint_name>front_left_wheel_joint</joint_name>
+            <joint_name>front_right_wheel_joint</joint_name>
+            <joint_name>rear_left_wheel_joint</joint_name>
+            <joint_name>rear_right_wheel_joint</joint_name>
+        </plugin>
+    </gazebo>
 </robot>

File: rover_description/urdf/skid_steer.urdf.xacro (robot description, xacro)
@@ -1,3 +1,3 @@
-<robot xmlns:xacro="http://ros.org/wiki/xacro">
+<robot xmlns:xacro="http://www.ros.org/wiki/xacro">
   <xacro:macro name="diff_drive_controller" params="wheel_separation wheel_radius">
     <gazebo>
